File: Micromouse/MicromouseSchematic/IR_Sensor.kicad_sch (KiCad schematic)
At the start: 7 parts, among them J12 IR_1, Q10 DMN3065LW-7, Q9 SFH300

Commit message: Afarnfa
Parts:
- Q10: footprint DMN3065LW-7 -> MM_DMN3065LW-7:DMN3065LW-7
Changed lines of the file:
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@@
 			)
 		)
-		(property "Footprint" "DMN3065LW-7"
+		(property "Footprint" "MM_DMN3065LW-7:DMN3065LW-7"
 			(at 143.51 68.58 0)
 			(effects
