File: Micromouse/MicromouseSchematic/IR_Sensor.kicad_sch (KiCad schematic)
At the start: 7 parts, among them J12 IR_1, Q10 DMN3065LW-7, Q9 SFH300

Commit message: integration: rename Daniel's IR J12 to J9 + KiCad annotation cleanup
Resolves a second reference-designator collision: Daniel's IR sensor
schematic (IR_Sensor.kicad_sch) used J12, but Aahan's motor-driver
schematic also defines a J12. Renamed Daniel's IR J12 -> J9 (J9 was a
free slot on origin/main since Daniel had previously removed an
ancestor component using that designator).

Also incorporates KiCad's auto-cleanup from Tools -> Annotate Schematic:
regenerated junction/wire UUIDs in the top-level schematic and
re-canonicalized track widths and text sizes in MicromouseSchematic.kicad_pro.
These are cosmetic file-format changes from KiCad opening and re-saving
the project after the J12->J9 rename.

Reference designators across the integration schematic are now unique:
J1-J14 with no duplicates. J13 = Ragbot's TOF connector (6-pin),
J14 = Aahan's motor driver connector (10-pin), J9 = Daniel's IR
connector (was J12).

PCB merge still pending: Append Board for Aahan's motor driver layout
and Ragbot's TOF layout, with a ghost-J9 cleanup since Aahan's PCB
contains a leftover J9 footprint inherited from the common ancestor
(not present in any of Aahan's schematic files).

Co-authored-by: Cursor <cursoragent@cursor.com>
Parts:
- renumbered J12 to J9
Changed lines of the file:
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@@
 		(on_board yes)
 		(dnp no)
-		(property "Reference" "#PWR016"
+		(property "Reference" "#PWR0102"
 			(at 107.95 110.49 0)
 			(effects
@@
 			(project "MicromouseSchematic"
 				(path "/0dcfab91-6b00-43c0-ac0b-8c301cb559e5/13f4247b-848d-475d-83d5-f2fff083c70d/13dfd103-1647-47ca-a8d4-32c9a2fd1e3b"
-					(reference "#PWR017")
-					(unit 1)
-				)
-				(path "/0dcfab91-6b00-43c0-ac0b-8c301cb559e5/13f4247b-848d-475d-83d5-f2fff083c70d/25d673b4-6a3b-4604-bba1-73aa25dddacb"
-					(reference "#PWR018")
-					(unit 1)
-				)
-				(path "/0dcfab91-6b00-43c0-ac0b-8c301cb559e5/13f4247b-848d-475d-83d5-f2fff083c70d/c3359d57-31d6-4e97-bb88-fe098e219bf4"
-					(reference "#PWR016")
+					(reference "#PWR0103")
+					(unit 1)
+				)
+				(path "/0dcfab91-6b00-43c0-ac0b-8c301cb559e5/13f4247b-848d-475d-83d5-f2fff083c70d/25d673b4-6a3b-4604-bba1-73aa25dddacb"
+					(reference "#PWR0104")
+					(unit 1)
+				)
+				(path "/0dcfab91-6b00-43c0-ac0b-8c301cb559e5/13f4247b-848d-475d-83d5-f2fff083c70d/c3359d57-31d6-4e97-bb88-fe098e219bf4"
+					(reference "#PWR0102")
 					(unit 1)
 				)
@@
 		(on_board yes)
 		(dnp no)
-		(property "Reference" "J12"
+		(property "Reference" "J9"
 			(at 82.296 79.248 0)
 			(effects
@@
 				)
 				(path "/0dcfab91-6b00-43c0-ac0b-8c301cb559e5/13f4247b-848d-475d-83d5-f2fff083c70d/c3359d57-31d6-4e97-bb88-fe098e219bf4"
-					(reference "J12")
-					(unit 1)
-				)
+					(reference "J9")
+					(unit 1)
+				)
