File: Micromouse/MicromouseSchematic/motordrivers.kicad_sch (KiCad schematic)
At the start: 19 parts, among them J1 Conn_01x06_MountingPin, J2 Conn_01x06_MountingPin, U11 MP6550GG-Z, U7 MP6550GG-Z

Commit message: integration: assemble sub-schematics from each contributor
Take motordrivers.kicad_sch from origin/aahan (Aahan's motor driver work)
and tof.kicad_sch from origin/ragbot/tof_changes (ToF sensor connector).
Daniel's IR_Sensor.kicad_sch and irsens.kicad_sch are inherited from the
origin/main baseline of this integration branch.

Renamed Aahan's J13 (Conn_01x10, motor-driver connector) to J14 to
resolve a reference-designator collision with Ragbot's J13 (Conn_01x06,
TOF sensor connector). Both connectors keep their respective UUIDs and
footprints; only the reference text changes.

The MicromouseSchematic.kicad_pcb still needs to be merged in KiCad via
File -> Append Board to bring in Aahan's motor-driver footprints and
Ragbot's TOF connector on top of Daniel's IR-focused base layout.

Co-authored-by: Cursor <cursoragent@cursor.com>
Parts:
- added Cin_MD2: 22 μF, Capacitor_SMD:C_0402_1005Metric, symbol Device:C
- added J12, J14: Conn_01x10, Connector_JST:JST_ZH_B10B-ZR_1x10_P1.50mm_Vertical, symbol Connector_Generic:Conn_01x10
Connections:
- net Encoder A (1): now also J14.8 (Pin_8)
- net Encoder A (2): now also J12.8 (Pin_8)
- net Encoder B (1): now also J14.7 (Pin_7)
- net Encoder B (2): now also J12.7 (Pin_7)
- net GND: now also Cin_MD2.2, J12.9 (Pin_9), J14.9 (Pin_9)
- net IN1(1): now also J14.4 (Pin_4)
- net IN1(2): now also J12.4 (Pin_4)
- net IN2(1): now also J14.5 (Pin_5)
- net IN2(2): now also J12.5 (Pin_5)
- net NSLEEP_HB(1): now also J14.2 (Pin_2)
- net NSLEEP_HB(2): now also J12.2 (Pin_2)
- net NSLEEP_LDO(1): now also J14.3 (Pin_3)
- net NSLEEP_LDO(2): now also J12.3 (Pin_3)
- net VCC: now also J12.1 (Pin_1), J14.1 (Pin_1)
- net VISEN(1): now also J14.6 (Pin_6)
- net VISEN(2): now also J12.6 (Pin_6)
- net Vin (7.4 V): now also Cin_MD2.1, J12.10 (Pin_10), J14.10 (Pin_10)
