File: Micromouse/MicromouseSchematic/MicromouseSchematic.kicad_pcb (KiCad board)
At the start: 2 copper layers, 155.7 x 48 mm, 105 parts, among them J1 Conn_01x06_MountingPin, J10 Conn_01x06_MountingPin, J11 Conn_01x07_Pin, J12 Conn_01x10, J13 Conn_01x06_Pin, J14 Conn_01x10, J2 Conn_01x06_MountingPin, J3 Conn_01x03_Pin, J4 Conn_01x02_Pin, J5 Conn_01x06_MountingPin, J6 IR_1, J7 IR_1, J8 IR_1, J9 IR_1, Q1 SFH300, Q10 DMN3065LW-7, Q2 DMN3065LW-7, Q3 SFH300, Q4 DMN3065LW-7, Q5 SFH300, Q6 DMN3065LW-7, Q9 SFH300, SW1 SW_Push, SW2 SW_Push, U1 VL53L1CXV0FY1, U11 MP6550GG-Z, U3 ICM-42688-P, U4 LIS2MDLTR, U5 STM32F746VETx, U7 MP6550GG-Z, Y1 8MHz, Y2 32.768kHz

Commit message: integration PCB: merge Aahan's motor driver + Ragbot's TOF layouts
Final PCB integration via two File -> Append Board operations
followed by Tools -> Update PCB from Schematic with orphan deletion:

1. Appended Aahan's PCB (kicad-merge-sources/aahan-pcb), then ran
   Update PCB from Schematic to:
   - Re-link Aahan's positioned motor-driver footprints (J12, J14,
     Cin_MD2, U7, U11, R40-R42, Renb1, Rent1, etc.) to the merged
     schematic symbols by reference designator.
   - Delete orphans: ancestor components Aahan kept but Daniel had
     intentionally removed (C41-C44, D4, J9 ghost, Q7, Q8, R25,
     R28-R34) and the duplicate origin-stacked footprints from the
     earlier Update PCB step.

2. Appended Ragbot's PCB (kicad-merge-sources/tof-pcb), then ran
   Update PCB from Schematic again with the same options to bring
   in Ragbot's TOF layout (J13 connector + supporting parts) and
   sweep any new orphans.

Plus minor manual placement / routing tweaks made by Ragbot in KiCad.

Cross-check after the merge:
- 106 unique footprints on the PCB.
- 106 unique reference designators in the merged schematic.
- Zero duplicate references on the PCB.
- Zero orphan footprints (every PCB footprint has a matching schematic
  symbol).
- Zero missing footprints (every schematic symbol has a matching PCB
  footprint).

Pre-existing issues that survive (not introduced by this merge):
- VR1 has 12 unconnected thermal/exposed pads (8-19) on the
  TPSM861253RDXR power module - typical for QFN packages.
- J1, J2, J5, J10 schematic symbols include an MP (Mounting Peg)
  pin that does not exist in the chosen JST footprint variants -
  flag for a future symbol/footprint cleanup pass.

kicad_pro: KiCad auto-added a GND netclass pattern next to the
existing +3.3V one. Cosmetic.

Co-authored-by: Cursor <cursoragent@cursor.com>
Parts:
- moved J13 120.9 mm to (103.5, 138.2), turned to -90 degrees
- moved J12 118.6 mm to (87.4, 84.2), turned to -90 degrees
- moved J14 98.0 mm to (87.8, 112.0), turned to -90 degrees
- moved Cin_MD2 82.3 mm to (81.8, 97.5), turned to 90 degrees
- moved R38 42.5 mm to (77.7, 119.5), turned to -90 degrees
- moved R37 42.4 mm to (78.1, 116.5)
- moved Cin_MD1 36.2 mm to (82.7, 125.0), turned to 90 degrees
- moved R42 36.1 mm to (83.1, 113.4), turned to 180 degrees
- moved J1 35.6 mm to (63.2, 115.0), turned to -90 degrees
- moved R41 33.9 mm to (78.2, 114.4)
- moved R40 31.9 mm to (82.7, 85.6), turned to 180 degrees
- moved U7 31.1 mm to (73.6, 118.0), turned to -90 degrees
- moved R21 30.9 mm to (71.2, 121.7), turned to -90 degrees
- moved C3 29.7 mm to (70.1, 119.2), turned to 180 degrees
- moved R35 28.3 mm to (77.8, 88.7)
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Routing:
- net GND: track 183.2 -> 328.6 mm, vias 12 -> 16
- net +3.3V: track 148.5 -> 288.1 mm
- net +7.4V: track 30.3 -> 66.3 mm
- net Encoder_B_1: track 0.00 -> 25.6 mm
- net Encoder_B_2: track 0.00 -> 25.6 mm
- net Encoder_A_1: track 0.00 -> 25.2 mm, vias 0 -> 1
- net Encoder_A_2: track 0.00 -> 25.2 mm, vias 0 -> 1
- net Net-(U11-NSLEEP_HB): track 0.00 -> 24.4 mm, vias 0 -> 2
- net MO2_IN2: track 0.00 -> 20.7 mm
- net TOF_CE: track 0.00 -> 18.2 mm, vias 0 -> 1
- net Net-(J2-Pin_2): track 0.00 -> 14.0 mm, vias 0 -> 1
- net Net-(J1-Pin_2): track 0.00 -> 14.0 mm, vias 0 -> 1
- net VISEN_1: track 0.00 -> 13.7 mm
- net VISEN_2: track 0.00 -> 13.7 mm
- net I2C_SDA: track 10.5 -> 24.1 mm, vias 0 -> 1
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- added copper zone on F.Cu, net GND
Other:
- board size 155.7 x 48 mm -> 155.7 x 131.7 mm
- board text added: "Driver 1"
- board text added: "Driver 2"
- board text removed: "Motor Drivers"
