File: Micromouse/Micromouse_main_project/voltagereg.kicad_sch (KiCad schematic)
At the start: 7 parts, among them U1 VL53L1CXV0FY1

Commit message: Schematic overhaul
Parts:
- removed C11: 100n, Capacitor_SMD:C_0402_1005Metric, symbol Device:C
- removed C9: 4.7u, Capacitor_SMD:C_0402_1005Metric, symbol Device:C
- removed R1, R2, R3, R4: 10k, Resistor_SMD:R_0603_1608Metric, symbol Device:R
- removed U1: VL53L1CXV0FY1, MM_VL53L4CDV0DH-1:LGA12_STM, symbol Sensor_Distance:VL53L1CXV0FY1
- added C22: 22u, Capacitor_SMD:C_0603_1608Metric, symbol Device:C
- added Cin_VR1: 10u, Capacitor_SMD:C_0603_1608Metric, symbol Device:C
- added Renb1: 30kΩ, Resistor_SMD:R_0603_1608Metric, symbol Device:R
- added Rent1: 62kΩ, Resistor_SMD:R_0603_1608Metric, symbol Device:R
- added VR1: TPSM861253RDXR, MM_TPSM861253RDXR:TPSM861253RDXR, symbol TPSM861253RDXR:TPSM861253RDXR
Connections:
- net GND: now also C22.2, Cin_VR1.2, Renb1.2, VR1.4 (PGND)
- new net: Renb1.1, Rent1.2, VR1.6 (EN)
- new net Vin(+7.4V): Cin_VR1.1, Rent1.1, VR1.1 (VIN)
- new net Vout(+3.3V): C22.1, VR1.3 (VOUT), VR1.7 (VOS)
- no-connect marks 0 -> 1
Other:
- note removed: "TOF 0"

Commit message: Prepped layout
Parts:
- VR1: footprint MM_TPSM861253RDXR:TPSM861253RDXR -> TPSM862253RDXR_FOOTPRINT:TPSM861253RDXR
Changed lines of the file:
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@@
 			)
 		)
-		(property "Footprint" "MM_TPSM861253RDXR:TPSM861253RDXR"
+		(property "Footprint" "TPSM862253RDXR_FOOTPRINT:TPSM861253RDXR"
 			(at 139.7 97.79 0)
 			(hide yes)

Commit message: Finished layout
Parts:
- renumbered C22 to C20
Changed lines of the file:
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@@
 		(dnp no)
 		(fields_autoplaced yes)
-		(property "Reference" "#PWR034"
+		(property "Reference" "#PWR035"
 			(at 161.29 114.3 0)
 			(hide yes)
@@
 			(project "MicromouseSchematic"
 				(path "/0dcfab91-6b00-43c0-ac0b-8c301cb559e5/3cd5e638-0450-45f9-91e1-d72f396e0d78"
-					(reference "#PWR034")
+					(reference "#PWR035")
 					(unit 1)
 				)
@@
 		(dnp no)
 		(fields_autoplaced yes)
-		(property "Reference" "#PWR032"
+		(property "Reference" "#PWR033"
 			(at 83.82 107.95 0)
 			(hide yes)
@@
 			(project "MicromouseSchematic"
 				(path "/0dcfab91-6b00-43c0-ac0b-8c301cb559e5/3cd5e638-0450-45f9-91e1-d72f396e0d78"
-					(reference "#PWR032")
+					(reference "#PWR033")
 					(unit 1)
 				)
@@
 		(dnp no)
 		(fields_autoplaced yes)
-		(property "Reference" "C22"
+		(property "Reference" "C20"
 			(at 173.99 95.2499 0)
 			(show_name no)
@@
 			(project "MicromouseSchematic"
 				(path "/0dcfab91-6b00-43c0-ac0b-8c301cb559e5/3cd5e638-0450-45f9-91e1-d72f396e0d78"
-					(reference "C22")
+					(reference "C20")
 					(unit 1)
 				)
@@
 		(dnp no)
 		(fields_autoplaced yes)
-		(property "Reference" "#PWR033"
+		(property "Reference" "#PWR034"
 			(at 106.68 113.03 0)
 			(hide yes)
@@
 			(project "MicromouseSchematic"
 				(path "/0dcfab91-6b00-43c0-ac0b-8c301cb559e5/3cd5e638-0450-45f9-91e1-d72f396e0d78"
-					(reference "#PWR033")
+					(reference "#PWR034")
 					(unit 1)
 				)
