File: Micromouse/Micromouse_main_project/MicromouseSchematic.kicad_sch (KiCad schematic)
At the start: 27 parts, among them J10 Conn_01x06_MountingPin, J4 Conn_01x02_Pin, J5 Conn_01x06_MountingPin, SW1 SW_Push, SW2 SW_Push, U5 STM32F746VETx, Y1 8MHz, Y2 32.768kHz

Commit message: Schematic overhaul
Parts:
- removed C28, C31: 6.8p, Capacitor_SMD:C_0402_1005Metric, symbol Device:C
- added C6, C7: 15p, Capacitor_SMD:C_0603_1608Metric, symbol Device:C
- added R2, R3: 3.3k, Resistor_SMD:R_0603_1608Metric, symbol Device:R
- C1: renamed from C20; value 10p -> 27p; footprint Capacitor_SMD:C_0402_1005Metric -> Capacitor_SMD:C_0603_1608Metric
- C10: renamed from C26; footprint Capacitor_SMD:C_0402_1005Metric -> Capacitor_SMD:C_0603_1608Metric
- C11: renamed from C27; footprint Capacitor_SMD:C_0402_1005Metric -> Capacitor_SMD:C_0603_1608Metric
- C12: renamed from C29; footprint Capacitor_SMD:C_0402_1005Metric -> Capacitor_SMD:C_0603_1608Metric
- C13: renamed from C30; footprint Capacitor_SMD:C_0402_1005Metric -> Capacitor_SMD:C_0603_1608Metric
- C14: renamed from C32; footprint Capacitor_SMD:C_0402_1005Metric -> Capacitor_SMD:C_0603_1608Metric
- C15: renamed from C33; footprint Capacitor_SMD:C_0402_1005Metric -> Capacitor_SMD:C_0603_1608Metric
- C16: renamed from C34; footprint Capacitor_SMD:C_0402_1005Metric -> Capacitor_SMD:C_0603_1608Metric
- C17: renamed from C35; footprint Capacitor_SMD:C_0402_1005Metric -> Capacitor_SMD:C_0603_1608Metric
- C2: renamed from C19; value 0.1u -> 100n; footprint Capacitor_SMD:C_0402_1005Metric -> Capacitor_SMD:C_0603_1608Metric
- C3: renamed from C21; value 10p -> 27p; footprint Capacitor_SMD:C_0402_1005Metric -> Capacitor_SMD:C_0603_1608Metric
- C4: renamed from C22; footprint Capacitor_SMD:C_0402_1005Metric -> Capacitor_SMD:C_0603_1608Metric
- C5: renamed from C23; footprint Capacitor_SMD:C_0402_1005Metric -> Capacitor_SMD:C_0603_1608Metric
- C8: renamed from C24; footprint Capacitor_SMD:C_0402_1005Metric -> Capacitor_SMD:C_0603_1608Metric
- C9: renamed from C25; footprint Capacitor_SMD:C_0402_1005Metric -> Capacitor_SMD:C_0603_1608Metric
- FB1: footprint Resistor_SMD:R_0805_2012Metric -> (none)
- renumbered J4 to J1, J10 to J2, J5 to J3, R20 to R1, U5 to U1
Connections:
- net +3.3V: now also R2.1, R3.1
- net GND: now also C1.1, C3.1, C6.2, C7.2
- net I2C_SCL: now also U1.95 (PB8), R2.2; no longer U1.96 (PB9)
- net I2C_SDA: now also U1.96 (PB9), R3.2; no longer U1.95 (PB8)
- net IMU_INT_1: now also U1.63 (PC6); no longer U1.16 (PC1)
- net IMU_INT_2: now also U1.64 (PC7); no longer U1.17 (PC2)
- net IR_REC_1: now also U1.15 (PC0); no longer U1.18 (PC3)
- net IR_REC_2: now also U1.16 (PC1); no longer U1.32 (PC4)
- net IR_REC_3: now also U1.17 (PC2); no longer U1.22 (PA0)
- net IR_REC_4: now also U1.18 (PC3); no longer U1.33 (PC5)
- net MAG_INT: now also U1.65 (PC8); no longer U1.15 (PC0)
- net at U1.12 (PH0): now also C1.2, Y1.1; no longer C1.1
- net at Y1.2: now also C3.2, U1.13 (PH1); no longer C3.1
- net at U1.8 (PC14): now also Y2.2, C7.1
- net at Y2.1: now also U1.9 (PC15), C6.1
- net TOF_SHUT1: now reaches U1.43 (PE13)
- net TOF_SHUT2: now reaches U1.44 (PE14)
- net TOF_SHUT3: now reaches U1.45 (PE15)
- net IMU_CS: now reaches U1.51 (PB12)
- net IMU_CLK: now reaches U1.52 (PB13)
- net IMU_MISO: now reaches U1.53 (PB14)
- net IMU_MOSI: now reaches U1.54 (PB15)
- net TOF_INT1: now reaches U1.66 (PC9)
- net MCU_TX: now reaches U1.68 (PA9)
- net MCU_TX: now also J3.5 (Pin_5)
- net MCU_RX: now reaches U1.69 (PA10)
- net MCU_RX: now also J3.4 (Pin_4)
- net TOF_INT2: now reaches U1.78 (PC10)
- net TOF_INT3: now reaches U1.79 (PC11)
- net RXD: no longer names the net of U1.86 (PD5)
- net RXD: no longer J3.5 (Pin_5)
- net TOF_CE: no longer names the net of U1.5 (PE6)
- net TOF_INT: no longer names the net of U1.7 (PC13)
- net TXD: no longer names the net of U1.87 (PD6)
- net TXD: no longer J3.4 (Pin_4)
- no-connect marks 45 -> 37
Other:
- sheet IMU and Magnetometer ports: added IMU_CLK, IMU_CS, IMU_MISO, IMU_MOSI, MAG_SCL, MAG_SDA; removed I2C_SCL, I2C_SDA
- sheet ToF ports: added INT1 (ToF), INT2 (ToF), INT3 (ToF), XSHUT1, XSHUT2, XSHUT3; removed CE, INT (ToF)
- note added: "3.3k pull-ups to ensure SDA & SCL rise fast for reliable 400 kHz I²C operation"
- note added: "MCU RX <- module TX MCU TX -> module RX"
- note added: "TODO: IMU & Mag, Bluetooth module, ToF, MCU pinouts, IR sensors"
- note removed: "TODO: Double check voltage regulator, IMU & Mag, Bluetooth module, crystal oscillator capacitor values, IR sensors, ToF, MCU pinouts"
- moved on the sheet: C1, C3, J1, J2, J3, Y2

Commit message: Prepped layout
Parts:
- FB1: footprint (none) -> Inductor_SMD:L_0603_1608Metric
- J2: footprint Connector_JST:JST_ZH_B6B-ZR_1x06_P1.50mm_Vertical -> Connector_PinHeader_2.54mm:PinHeader_1x06_P2.54mm_Vertical
- J3: footprint Connector_JST:JST_ZH_B6B-ZR_1x06_P1.50mm_Vertical -> Connector_PinSocket_2.54mm:PinSocket_1x06_P2.54mm_Vertical
- SW1, SW2: footprint Button_Switch_THT:SW_SPST_Omron_B3F-40xx -> Button_Switch_SMD:SW_SPST_SKQG_WithStem
Changed lines of the file:
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@@
 			)
 		)
-		(property "Footprint" "Connector_JST:JST_ZH_B6B-ZR_1x06_P1.50mm_Vertical"
+		(property "Footprint" "Connector_PinSocket_2.54mm:PinSocket_1x06_P2.54mm_Vertical"
 			(at 153.67 153.67 0)
 			(hide yes)
@@
 			)
 		)
-		(property "Footprint" "Button_Switch_THT:SW_SPST_Omron_B3F-40xx"
+		(property "Footprint" "Button_Switch_SMD:SW_SPST_SKQG_WithStem"
 			(at 21.59 40.64 0)
 			(hide yes)
@@
 			)
 		)
-		(property "Footprint" ""
+		(property "Footprint" "Inductor_SMD:L_0603_1608Metric"
 			(at 191.77 28.448 90)
 			(hide yes)
@@
 			)
 		)
-		(property "Footprint" "Button_Switch_THT:SW_SPST_Omron_B3F-40xx"
+		(property "Footprint" "Button_Switch_SMD:SW_SPST_SKQG_WithStem"
 			(at 41.91 40.64 0)
 			(hide yes)
@@
 			)
 		)
-		(property "Footprint" "Connector_JST:JST_ZH_B6B-ZR_1x06_P1.50mm_Vertical"
+		(property "Footprint" "Connector_PinHeader_2.54mm:PinHeader_1x06_P2.54mm_Vertical"
 			(at 139.7 72.39 0)
 			(hide yes)

Commit message: Finished layout
Connections:
- net NSLEEP_LDO_1: no longer names the net of U1.38 (PE8)
- net NSLEEP_LDO_2: no longer names the net of U1.42 (PE12)
- no-connect marks 37 -> 39
Other:
- sheet Motor Drivers ports: added none; removed NSLEEP_LDO(1), NSLEEP_LDO(2)
Changed lines of the file:
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@@
 	)
 	(no_connect
+		(at 49.53 85.09)
+	)
+	(no_connect
+		(at 49.53 95.25)
+	)
+	(no_connect
 		(at 49.53 115.57)
 	)
@@
 	(wire
 		(pts
-			(xy 261.62 106.68) (xy 264.16 106.68)
-		)
-		(stroke
-			(width 0)
-			(type default)
-		)
-	)
-	(wire
-		(pts
 			(xy 46.99 97.79) (xy 49.53 97.79)
 		)
@@
 	(wire
 		(pts
-			(xy 46.99 85.09) (xy 49.53 85.09)
-		)
-		(stroke
-			(width 0)
-			(type default)
-		)
-	)
-	(wire
-		(pts
 			(xy 226.06 91.44) (xy 228.6 91.44)
 		)
@@
 	(wire
 		(pts
-			(xy 226.06 106.68) (xy 228.6 106.68)
-		)
-		(stroke
-			(width 0)
-			(type default)
-		)
-	)
-	(wire
-		(pts
 			(xy 26.67 34.29) (xy 26.67 35.56)
 		)
@@
 	(wire
 		(pts
-			(xy 46.99 95.25) (xy 49.53 95.25)
-		)
-		(stroke
-			(width 0)
-			(type default)
-		)
-	)
-	(wire
-		(pts
 			(xy 160.02 34.29) (xy 168.91 34.29)
 		)
@@
 		)
 	)
-	(global_label "NSLEEP_LDO_2"
-		(shape input)
-		(at 264.16 106.68 0)
-		(fields_autoplaced yes)
-		(effects
-			(font
-				(size 1.27 1.27)
-			)
-			(justify left)
-		)
-		(property "Intersheetrefs" "${INTERSHEET_REFS}"
-			(at 281.0546 106.68 0)
-			(hide yes)
-			(show_name no)
-			(do_not_autoplace no)
-			(effects
-				(font
-					(size 1.27 1.27)
-				)
-				(justify left)
-			)
-		)
-	)
 	(global_label "IR_POW_4"
 		(shape input)
@@
 		)
 	)
-	(global_label "NSLEEP_LDO_2"
-		(shape input)
-		(at 46.99 95.25 180)
-		(fields_autoplaced yes)
-		(effects
-			(font
-				(size 1.27 1.27)
-			)
-			(justify right)
-		)
-		(property "Intersheetrefs" "${INTERSHEET_REFS}"
-			(at 30.0954 95.25 0)
-			(hide yes)
-			(show_name no)
-			(do_not_autoplace no)
-			(effects
-				(font
-					(size 1.27 1.27)
-				)
-				(justify right)
-			)
-		)
-	)
 	(global_label "IR_POW_1"
 		(shape input)
@@
 		)
 	)
-	(global_label "NSLEEP_LDO_1"
-		(shape input)
-		(at 46.99 85.09 180)
-		(fields_autoplaced yes)
-		(effects
-			(font
-				(size 1.27 1.27)
-			)
-			(justify right)
-		)
-		(property "Intersheetrefs" "${INTERSHEET_REFS}"
-			(at 30.0954 85.09 0)
-			(hide yes)
-			(show_name no)
-			(do_not_autoplace no)
-			(effects
-				(font
-					(size 1.27 1.27)
-				)
-				(justify right)
-			)
-		)
-	)
 	(global_label "IMU_CLK"
 		(shape input)
@@
 		)
 	)
-	(global_label "NSLEEP_LDO_1"
-		(shape input)
-		(at 226.06 106.68 180)
-		(fields_autoplaced yes)
-		(effects
-			(font
-				(size 1.27 1.27)
-			)
-			(justify right)
-		)
-		(property "Intersheetrefs" "${INTERSHEET_REFS}"
-			(at 209.1654 106.68 0)
-			(hide yes)
-			(show_name no)
-			(do_not_autoplace no)
-			(effects
-				(font
-					(size 1.27 1.27)
-				)
-				(justify right)
-			)
-		)
-	)
 	(global_label "Encoder_B_1"
 		(shape output)
@@
 	(sheet
 		(at 228.6 67.31)
-		(size 33.02 43.18)
+		(size 33.02 38.1)
 		(exclude_from_sim no)
 		(in_bom yes)
@@
 		)
 		(property "Sheetfile" "motordrivers.kicad_sch"
-			(at 228.6 111.0746 0)
+			(at 228.6 105.9946 0)
 			(show_name no)
 			(do_not_autoplace no)
@@
 			(effects
 				(font
-					(size 1.27 1.27)
-				)
-				(justify left)
-			)
-		)
-		(pin "NSLEEP_LDO(2)" input
-			(at 261.62 106.68 0)
-			(effects
-				(font
-					(size 1.27 1.27)
-				)
-				(justify right)
-			)
-		)
-		(pin "NSLEEP_LDO(1)" input
-			(at 228.6 106.68 180)
-			(effects
-				(font

Commit message: Completed IR board, ToF board, changed IMU
Parts:
- added D1: LED, LED_SMD:LED_0603_1608Metric, symbol Device:LED
- added R12: 330, Resistor_SMD:R_0603_1608Metric, symbol Device:R
- J1: footprint Connector_JST:JST_PH_B2B-PH-K_1x02_P2.00mm_Vertical -> Connector_Wire:SolderWire-2.5sqmm_1x02_P7.2mm_D2.4mm_OD3.6mm_Relief
- Y1: footprint Crystal:Crystal_SMD_5032-2Pin_5.0x3.2mm -> MM_8MHz:XTAL_ECS-80-18-30-JGN-TR
- Y2: footprint Crystal:Crystal_SMD_3215-2Pin_3.2x1.5mm -> MM_32.7kHz:XTAL_ECS-31B_ECS
Connections:
- net GND: now also D1.1 (K)
- net TEST_LED: now reaches U1.34 (PB0)
- net TEST_LED: now also R12.1
- new net: D1.2 (A), R12.2
- no-connect marks 39 -> 38
Other:
- note added: "VISEN = current draw as an analog voltage"
- note removed: "TODO: IMU & Mag, Bluetooth module, ToF, MCU pinouts, IR sensors"
